File: FullSchematic/FullSchematic/AnalogueSensor.sch (KiCad schematic (older format))
At the start: 2 parts

Commit message: Combing all schematics
Parts:
- renumbered R1 to R?, R2 to R?
Connections:
- net Vout renamed LDR
Changed lines of the file:
@@
 $Descr A4 11693 8268
 encoding utf-8
-Sheet 1 1
+Sheet 2 3
 Title "Analogue Sensor"
 Date "2023-03-04"
@@
 Vcc
 $Comp
-L Device:R_Small R1
+L Device:R_Small R?
 U 1 1 640358D9
 P 3200 2300
-F 0 "R1" H 3259 2346 50  0000 L CNN
+F 0 "R?" H 3259 2346 50  0000 L CNN
 F 1 "180" H 3259 2255 50  0000 L CNN
 F 2 "Resistor_SMD:R_0201_0603Metric" H 3200 2300 50  0001 C CNN
@@
 $EndComp
 $Comp
-L Sensor_Optical:LDR03 R2
+L Sensor_Optical:LDR03 R?
 U 1 1 640363B3
 P 3200 3100
-F 0 "R2" H 3270 3146 50  0000 L CNN
+F 0 "R?" H 3270 3146 50  0000 L CNN
 F 1 "LDR03" H 3270 3055 50  0000 L CNN
 F 2 "OptoDevice:R_LDR_10x8.5mm_P7.6mm_Vertical" V 3375 3100 50  0001 C CNN
@@
 	3200 2400 3200 2700
 $Comp
-L power:GND #PWR0101
+L power:GND #PWR?
 U 1 1 64036F9E
 P 3200 3250
-F 0 "#PWR0101" H 3200 3000 50  0001 C CNN
+F 0 "#PWR?" H 3200 3000 50  0001 C CNN
 F 1 "GND" H 3205 3077 50  0000 C CNN
 F 2 "" H 3200 3250 50  0001 C CNN
@@
 	1    0    0    -1
 $EndComp
-Text GLabel 4050 2700 2    50   Input ~ 0
-Vout
 Wire Wire Line
 	3200 2700 4050 2700
@@
 Wire Wire Line
 	3200 2700 3200 2950
+Text HLabel 4050 2700 2    50   Input ~ 0
+LDR
 $EndSCHEMATC
