File: FullSchematic/FullSchematic/DigitalSensor.sch (KiCad schematic (older format))
At the start: 3 parts, among them IC1 TTP223E-BA6

Commit message: Combing all schematics
Parts:
- renumbered C1 to C?, C2 to C?, IC1 to IC?
Connections:
- net Output renamed T-Sensor
Changed lines of the file:
@@
 $Descr A4 11693 8268
 encoding utf-8
-Sheet 1 1
+Sheet 3 3
 Title "Digital Sensor"
 Date "2023-03-04"
@@
 $EndDescr
 $Comp
-L TTP223E-BA6:TTP223E-BA6 IC1
+L TTP223E-BA6:TTP223E-BA6 IC?
 U 1 1 64037076
 P 5450 3750
-F 0 "IC1" H 6000 4015 50  0000 C CNN
+F 0 "IC?" H 6000 4015 50  0000 C CNN
 F 1 "TTP223E-BA6" H 6000 3924 50  0000 C CNN
 F 2 "TTP223E-BA6:SOT95P285X126-6N" H 6400 3850 50  0001 L CNN
@@
 	6700 3750 6700 3850
 $Comp
-L pspice:CAP C1
+L pspice:CAP C?
 U 1 1 64038F20
 P 6700 4650
-F 0 "C1" H 6878 4696 50  0000 L CNN
+F 0 "C?" H 6878 4696 50  0000 L CNN
 F 1 "100n" H 6878 4605 50  0000 L CNN
 F 2 "Capacitor_THT:CP_Axial_L10.0mm_D4.5mm_P15.00mm_Horizontal" H 6700 4650 50  0001 C CNN
@@
 	6700 4950 6700 4900
 $Comp
-L power:GND #PWR0101
+L power:GND #PWR?
 U 1 1 6403A742
 P 5100 4950
-F 0 "#PWR0101" H 5100 4700 50  0001 C CNN
+F 0 "#PWR?" H 5100 4700 50  0001 C CNN
 F 1 "GND" H 5105 4777 50  0000 C CNN
 F 2 "" H 5100 4950 50  0001 C CNN
@@
 Wire Wire Line
 	4650 3650 5200 3650
-Text GLabel 4950 3350 0    50   Input ~ 0
-Output
 Wire Wire Line
 	4950 3350 5350 3350
@@
 	5350 3750 5450 3750
 $Comp
-L Device:C_Variable C2
+L Device:C_Variable C?
 U 1 1 64049E25
 P 4550 4100
-F 0 "C2" H 4665 4146 50  0000 L CNN
+F 0 "C?" H 4665 4146 50  0000 L CNN
 F 1 "C_Variable" H 4665 4055 50  0000 L CNN
 F 2 "Capacitor_SMD:C_Trimmer_Murata_TZC3" H 4550 4100 50  0001 C CNN
@@
 Wire Wire Line
 	4550 4250 4550 4700
+Text HLabel 4950 3350 0    50   Input ~ 0
+T-Sensor
 $EndSCHEMATC
