File: FullSchematic/FullSchematic/AnalogueSensor.kicad_sch (KiCad schematic)
At the start: 5 parts

Commit message: Aimee
Parts:
- R?: footprint OptoDevice:R_LDR_7x6mm_P5.1mm_Vertical -> OptoDevice:R_LDR_10x8.5mm_P7.6mm_Vertical
Changed lines of the file:
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@@
       (effects (font (size 1.27 1.27)) (justify left))
     )
-    (property "Footprint" "OptoDevice:R_LDR_7x6mm_P5.1mm_Vertical" (at 85.725 78.74 90)
+    (property "Footprint" "OptoDevice:R_LDR_10x8.5mm_P7.6mm_Vertical" (at 85.725 78.74 90)
       (effects (font (size 1.27 1.27)) hide)
     )

Commit message: added more footprints
Parts:
- R?: footprint OptoDevice:R_LDR_10x8.5mm_P7.6mm_Vertical -> OptoDevice:R_LDR_7x6mm_P5.1mm_Vertical
Changed lines of the file:
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@@
       (effects (font (size 1.27 1.27)) (justify left))
     )
-    (property "Footprint" "OptoDevice:R_LDR_10x8.5mm_P7.6mm_Vertical" (at 85.725 78.74 90)
+    (property "Footprint" "OptoDevice:R_LDR_7x6mm_P5.1mm_Vertical" (at 85.725 78.74 90)
       (effects (font (size 1.27 1.27)) hide)
     )
