File: FullSchematic/FullSchematic/AnalogueSensor.kicad_sch (KiCad schematic)
At the start: 5 parts

Commit message: resetting
Parts:
- TP10, TP8, TP9: footprint (none) -> TestPoint:TestPoint_Pad_D2.0mm
Changed lines of the file:
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@@
       (effects (font (size 1.27 1.27)))
     )
-    (property "Footprint" "" (at 81.28 58.42 0)
+    (property "Footprint" "TestPoint:TestPoint_Pad_D2.0mm" (at 81.28 58.42 0)
       (effects (font (size 1.27 1.27)) hide)
     )
@@
       (effects (font (size 1.27 1.27)))
     )
-    (property "Footprint" "" (at 81.28 67.31 0)
+    (property "Footprint" "TestPoint:TestPoint_Pad_D2.0mm" (at 81.28 67.31 0)
       (effects (font (size 1.27 1.27)) hide)
     )
@@
       (effects (font (size 1.27 1.27)) (justify left))
     )
-    (property "Footprint" "" (at 97.79 68.58 0)
+    (property "Footprint" "TestPoint:TestPoint_Pad_D2.0mm" (at 97.79 68.58 0)
       (effects (font (size 1.27 1.27)) hide)
     )

Commit message: Opening MicroController
Parts:
- TP10, TP8, TP9: footprint TestPoint:TestPoint_Pad_D2.0mm -> (none)
Changed lines of the file:
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@@
       (effects (font (size 1.27 1.27)))
     )
-    (property "Footprint" "TestPoint:TestPoint_Pad_D2.0mm" (at 81.28 58.42 0)
+    (property "Footprint" "" (at 81.28 58.42 0)
       (effects (font (size 1.27 1.27)) hide)
     )
@@
       (effects (font (size 1.27 1.27)))
     )
-    (property "Footprint" "TestPoint:TestPoint_Pad_D2.0mm" (at 81.28 67.31 0)
+    (property "Footprint" "" (at 81.28 67.31 0)
       (effects (font (size 1.27 1.27)) hide)
     )
@@
       (effects (font (size 1.27 1.27)) (justify left))
     )
-    (property "Footprint" "TestPoint:TestPoint_Pad_D2.0mm" (at 97.79 68.58 0)
+    (property "Footprint" "" (at 97.79 68.58 0)
       (effects (font (size 1.27 1.27)) hide)
     )
