File: FullSchematic/FullSchematic/DigitalSensor.kicad_sch (KiCad schematic)
At the start: 7 parts

Commit message: Aimee
Parts:
- TP13: footprint TestPoint:TestPoint_Pad_D2.0mm -> (none)
Changed lines of the file:
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@@
       (effects (font (size 1.27 1.27)) (justify left))
     )
-    (property "Footprint" "TestPoint:TestPoint_Pad_D2.0mm" (at 143.51 95.25 0)
+    (property "Footprint" "" (at 143.51 95.25 0)
       (effects (font (size 1.27 1.27)) hide)
     )

Commit message: added more footprints
Parts:
- TP13: footprint (none) -> TestPoint:TestPoint_Pad_D2.0mm
Changed lines of the file:
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@@
       (effects (font (size 1.27 1.27)) (justify left))
     )
-    (property "Footprint" "" (at 143.51 95.25 0)
+    (property "Footprint" "TestPoint:TestPoint_Pad_D2.0mm" (at 143.51 95.25 0)
       (effects (font (size 1.27 1.27)) hide)
     )
