File: FullSchematic/FullSchematic/DigitalSensor.kicad_sch (KiCad schematic)
At the start: 7 parts

Commit message: completed and generated BOM
Parts:
- C?: Price 0.0009 -> 0.08; Price ( 1 board) 0.0009 -> 0.32; Price (5 boards) 0.0045 -> 1.6
Changed lines of the file:
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@@
       (effects (font (size 1.27 1.27)) hide)
     )
-    (property "Price" "0.0009" (at 170.18 118.11 0)
+    (property "Price" "0.08" (at 170.18 118.11 0)
       (effects (font (size 1.27 1.27)) hide)
     )
-    (property "Price ( 1 board)" "0.0009" (at 170.18 118.11 0)
+    (property "Price ( 1 board)" "0.32" (at 170.18 118.11 0)
       (effects (font (size 1.27 1.27)) hide)
     )
-    (property "Price (5 boards)" "0.0045" (at 170.18 118.11 0)
+    (property "Price (5 boards)" "1.6" (at 170.18 118.11 0)
       (effects (font (size 1.27 1.27)) hide)
     )

Commit message: resetting
Parts:
- TP11, TP12, TP14: footprint (none) -> TestPoint:TestPoint_Pad_D2.0mm
Changed lines of the file:
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@@
       (effects (font (size 1.27 1.27)) (justify left))
     )
-    (property "Footprint" "" (at 110.49 97.79 0)
+    (property "Footprint" "TestPoint:TestPoint_Pad_D2.0mm" (at 110.49 97.79 0)
       (effects (font (size 1.27 1.27)) hide)
     )
@@
       (effects (font (size 1.27 1.27)) (justify right))
     )
-    (property "Footprint" "" (at 162.56 97.79 0)
+    (property "Footprint" "TestPoint:TestPoint_Pad_D2.0mm" (at 162.56 97.79 0)
       (effects (font (size 1.27 1.27)) hide)
     )
@@
       (effects (font (size 1.27 1.27)) (justify left))
     )
-    (property "Footprint" "" (at 172.72 95.25 0)
+    (property "Footprint" "TestPoint:TestPoint_Pad_D2.0mm" (at 172.72 95.25 0)
       (effects (font (size 1.27 1.27)) hide)
     )

Commit message: Opening MicroController
Parts:
- TP11, TP12, TP14: footprint TestPoint:TestPoint_Pad_D2.0mm -> (none)
Changed lines of the file:
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@@
       (effects (font (size 1.27 1.27)) (justify left))
     )
-    (property "Footprint" "TestPoint:TestPoint_Pad_D2.0mm" (at 110.49 97.79 0)
+    (property "Footprint" "" (at 110.49 97.79 0)
       (effects (font (size 1.27 1.27)) hide)
     )
@@
       (effects (font (size 1.27 1.27)) (justify right))
     )
-    (property "Footprint" "TestPoint:TestPoint_Pad_D2.0mm" (at 162.56 97.79 0)
+    (property "Footprint" "" (at 162.56 97.79 0)
       (effects (font (size 1.27 1.27)) hide)
     )
@@
       (effects (font (size 1.27 1.27)) (justify left))
     )
-    (property "Footprint" "TestPoint:TestPoint_Pad_D2.0mm" (at 172.72 95.25 0)
+    (property "Footprint" "" (at 172.72 95.25 0)
       (effects (font (size 1.27 1.27)) hide)
     )
