File: FullSchematic/FullSchematic/DigitalSensor.kicad_sch (KiCad schematic)
At the start: 7 parts

Commit message: updated schematic and footprints
Parts:
- IC?: footprint TTP223E-BA6:SOT95P285X126-6N -> Package_TO_SOT_SMD:SOT-563
Changed lines of the file:
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@@
       (effects (font (size 1.27 1.27)))
     )
-    (property "Footprint" "TTP223E-BA6:SOT95P285X126-6N" (at 162.56 92.71 0)
+    (property "Footprint" "Package_TO_SOT_SMD:SOT-563" (at 162.56 92.71 0)
       (effects (font (size 1.27 1.27)) (justify left) hide)
     )

Commit message: connected sensors adnd created touch pad
Parts:
- added P1: ~, Library:Touch Pad, symbol UCT:TouchPad
Connections:
- net Touch Pad: no longer names the net of C?.1, IC?.3 (I), TP14.1
- net Touch Pad: now also P1. (IN)
Changed lines of the file:
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@@
   (junction (at 170.18 95.25) (diameter 0) (color 0 0 0 0)
+  )
+  (junction (at 101.727 97.79) (diameter 0) (color 0 0 0 0)
   )
   (junction (at 129.54 125.73) (diameter 0) (color 0 0 0 0)
@@
     (stroke (width 0) (type default))
   )
-  (wire (pts (xy 101.6 97.79) (xy 105.41 97.79))
+  (wire (pts (xy 101.6 97.79) (xy 101.727 97.79))
     (stroke (width 0) (type default))
   )
@@
     (stroke (width 0) (type default))
   )
+  (wire (pts (xy 101.727 97.79) (xy 105.41 97.79))
+    (stroke (width 0) (type default))
+  )
   (wire (pts (xy 170.18 111.76) (xy 170.18 97.79))
     (stroke (width 0) (type default))
@@
   (wire (pts (xy 170.18 95.25) (xy 167.64 95.25))
     (stroke (width 0) (type default))
-  )
-  (label "Touch Pad" (at 101.6 97.79 180) (fields_autoplaced)
-    (effects (font (size 1.27 1.27)) (justify right bottom))
   )
   (hierarchical_label "T_sensor" (shape input) (at 125.73 85.09 180) (fields_autoplaced)
@@
         )
       )
+    )
+  )
+  (symbol (lib_id "UCT:TouchPad") (at 95.377 99.06 0) (unit 1)
+    (in_bom yes) (on_board yes) (dnp no) (fields_autoplaced)
+    (property "Reference" "P1" (at 102.9915 88.9 0)
+      (effects (font (size 1.27 1.27)))
+    )
+    (property "Value" "~" (at 95.377 99.06 0)
+      (effects (font (size 1.27 1.27)))
+    )
+    (property "Footprint" "Library:Touch Pad" (at 95.377 99.06 0)
+      (effects (font (size 1.27 1.27)) hide)
+    )
+    (property "Datasheet" "" (at 95.377 99.06 0)
+      (effects (font (size 1.27 1.27)) hide)
+    )
+    (pin "")
+    (instances
+      (project "FullSchematic"
+        (path "/5dd86611-a33d-45ee-946c-01c599f30b12/ef09fc32-79b3-4972-8ce2-fc52eddbfbb8/00000000-0000-0000-0000-0000640c1ec4"
+          (reference "P1") (unit 1)
+        )
+      )
