File: FullSchematic/FullSchematic/Microcontroller Schematic.kicad_sch (KiCad schematic)
At the start: 30 parts, among them J1 USB_B_Micro, J3 Conn_01x24_Socket, J4 Conn_01x24_Socket, U2 FT231XS, U3 24LC64

Commit message: added more footprints
Parts:
- R1, R2, R3, R6: footprint (none) -> Resistor_SMD:R_0201_0603Metric
- TP1, TP2, TP3, TP4, TP5, TP6, TP7: footprint (none) -> TestPoint:TestPoint_Pad_D2.0mm
Changed lines of the file:
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@@
       (effects (font (size 1.27 1.27)) (justify left))
     )
-    (property "Footprint" "" (at 62.23 46.99 0)
+    (property "Footprint" "TestPoint:TestPoint_Pad_D2.0mm" (at 62.23 46.99 0)
       (effects (font (size 1.27 1.27)) hide)
     )
@@
       (effects (font (size 1.27 1.27)))
     )
-    (property "Footprint" "" (at 155.194 113.284 90)
+    (property "Footprint" "Resistor_SMD:R_0201_0603Metric" (at 155.194 113.284 90)
       (effects (font (size 1.27 1.27)) hide)
     )
@@
       (effects (font (size 1.27 1.27)) (justify left))
     )
-    (property "Footprint" "" (at 166.37 132.08 0)
+    (property "Footprint" "TestPoint:TestPoint_Pad_D2.0mm" (at 166.37 132.08 0)
       (effects (font (size 1.27 1.27)) hide)
     )
@@
       (effects (font (size 1.27 1.27)))
     )
-    (property "Footprint" "" (at 155.194 131.064 90)
+    (property "Footprint" "Resistor_SMD:R_0201_0603Metric" (at 155.194 131.064 90)
       (effects (font (size 1.27 1.27)) hide)
     )
@@
       (effects (font (size 1.27 1.27)) (justify left))
     )
-    (property "Footprint" "" (at 167.64 114.3 0)
+    (property "Footprint" "TestPoint:TestPoint_Pad_D2.0mm" (at 167.64 114.3 0)
       (effects (font (size 1.27 1.27)) hide)
     )
@@
       (effects (font (size 1.27 1.27)))
     )
-    (property "Footprint" "" (at 155.194 122.174 90)
+    (property "Footprint" "Resistor_SMD:R_0201_0603Metric" (at 155.194 122.174 90)
       (effects (font (size 1.27 1.27)) hide)
     )
@@
       (effects (font (size 1.27 1.27)) (justify right))
     )
-    (property "Footprint" "" (at 74.93 166.37 0)
+    (property "Footprint" "TestPoint:TestPoint_Pad_D2.0mm" (at 74.93 166.37 0)
       (effects (font (size 1.27 1.27)) hide)
     )
@@
       (effects (font (size 1.27 1.27)) (justify left))
     )
-    (property "Footprint" "" (at 160.02 44.45 0)
+    (property "Footprint" "TestPoint:TestPoint_Pad_D2.0mm" (at 160.02 44.45 0)
       (effects (font (size 1.27 1.27)) hide)
     )
@@
       (effects (font (size 1.27 1.27)))
     )
-    (property "Footprint" "" (at 69.596 42.926 90)
+    (property "Footprint" "Resistor_SMD:R_0201_0603Metric" (at 69.596 42.926 90)
       (effects (font (size 1.27 1.27)) hide)
     )
@@
       (effects (font (size 1.27 1.27)) (justify left))
     )
-    (property "Footprint" "" (at 167.64 123.19 0)
+    (property "Footprint" "TestPoint:TestPoint_Pad_D2.0mm" (at 167.64 123.19 0)
       (effects (font (size 1.27 1.27)) hide)
     )
@@
       (effects (font (size 1.27 1.27)) (justify left))
     )
-    (property "Footprint" "" (at 77.47 69.85 0)
-      (effects (font (size 1.27 1.27)) hide)
-    )
+    (property "Footprint" "TestPoint:TestPoint_Pad_D2.0mm" (at 77.47 69.85 0)
+      (effects (font (size 1.27 1.27)) hide)
+    )

Commit message: Before merge-aimee
Parts:
- J1: footprint (none) -> SpecificFootprints:MICROXNJ
Changed lines of the file:
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@@
       (effects (font (size 1.27 1.27)))
     )
-    (property "Footprint" "" (at 134.62 59.69 0)
+    (property "Footprint" "SpecificFootprints:MICROXNJ" (at 134.62 59.69 0)
       (effects (font (size 1.27 1.27)) hide)
     )
