File: FullSchematic/FullSchematic/Power module.kicad_sch (KiCad schematic)
At the start: 1 part

Commit message: added more footprints
Parts:
- BT1: footprint (none) -> SpecificFootprints:BH18650PC; JLCPCB Part # (none) -> C2988620; Price (none) -> $1.31; Price ( 1 board) (none) -> $1.31; Price (5 boards) (none) -> 6.55
Changed lines of the file:
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@@
       (effects (font (size 1.27 1.27)) (justify left))
     )
-    (property "Footprint" "" (at 154.94 79.756 90)
+    (property "Footprint" "SpecificFootprints:BH18650PC" (at 154.94 79.756 90)
       (effects (font (size 1.27 1.27)) hide)
     )
@@
       (effects (font (size 1.27 1.27)) hide)
     )
-    (property "Price ( 1 board)" "" (at 154.94 81.28 0)
+    (property "Price ( 1 board)" "$1.31" (at 154.94 81.28 0)
       (effects (font (size 1.27 1.27)) hide)
     )
-    (property "Price (5 boards)" "" (at 154.94 81.28 0)
+    (property "Price (5 boards)" "6.55" (at 154.94 81.28 0)
       (effects (font (size 1.27 1.27)) hide)
     )
+    (property "JLCPCB Part #" "C2988620" (at 154.94 81.28 0)
+      (effects (font (size 1.27 1.27)) hide)
+    )
+    (property "Price" "$1.31" (at 154.94 81.28 0)
+      (effects (font (size 1.27 1.27)) hide)
+    )

Commit message: Aimee
Parts:
- BT1: footprint SpecificFootprints:BH18650PC -> (none); JLCPCB Part # C2988620 -> (none); Price $1.31 -> (none); Price ( 1 board) $1.31 -> (none); Price (5 boards) 6.55 -> (none)
Changed lines of the file:
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@@
       (effects (font (size 1.27 1.27)) (justify left))
     )
-    (property "Footprint" "SpecificFootprints:BH18650PC" (at 154.94 79.756 90)
+    (property "Footprint" "" (at 154.94 79.756 90)
       (effects (font (size 1.27 1.27)) hide)
     )
@@
       (effects (font (size 1.27 1.27)) hide)
     )
-    (property "Price ( 1 board)" "$1.31" (at 154.94 81.28 0)
+    (property "Price ( 1 board)" "" (at 154.94 81.28 0)
       (effects (font (size 1.27 1.27)) hide)
     )
-    (property "Price (5 boards)" "6.55" (at 154.94 81.28 0)
+    (property "Price (5 boards)" "" (at 154.94 81.28 0)
       (effects (font (size 1.27 1.27)) hide)
     )
-    (property "JLCPCB Part #" "C2988620" (at 154.94 81.28 0)
-      (effects (font (size 1.27 1.27)) hide)
-    )
-    (property "Price" "$1.31" (at 154.94 81.28 0)
-      (effects (font (size 1.27 1.27)) hide)
-    )
