File: FullSchematic/FullSchematic/Power module.kicad_sch (KiCad schematic)
At the start: 1 part

Commit message: adding of all footprints
Parts:
- BT1: footprint (none) -> Library:BH18650PC
Changed lines of the file:
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@@
       (effects (font (size 1.27 1.27)) (justify left))
     )
-    (property "Footprint" "" (at 154.94 79.756 90)
+    (property "Footprint" "Library:BH18650PC" (at 154.94 79.756 90)
       (effects (font (size 1.27 1.27)) hide)
     )
