File: FullSchematic/FullSchematic/Power module.kicad_sch (KiCad schematic)
At the start: 1 part

Commit message: updated schematics and footprints
Parts:
- BT1: footprint Library:BH18650PC -> Battery:BatteryHolder_Keystone_1042_1x18650; JLCPCB Part # (none) -> C2988620; Price (none) -> 1.41; Price ( 1 board) (none) -> 1.41; Price (5 boards) (none) -> 7.05
Changed lines of the file:
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@@
       (effects (font (size 1.27 1.27)) (justify left))
     )
-    (property "Footprint" "Library:BH18650PC" (at 154.94 79.756 90)
+    (property "Footprint" "Battery:BatteryHolder_Keystone_1042_1x18650" (at 154.94 79.756 90)
       (effects (font (size 1.27 1.27)) hide)
     )
@@
       (effects (font (size 1.27 1.27)) hide)
     )
-    (property "Price ( 1 board)" "" (at 154.94 81.28 0)
+    (property "Price ( 1 board)" "1.41" (at 154.94 81.28 0)
       (effects (font (size 1.27 1.27)) hide)
     )
-    (property "Price (5 boards)" "" (at 154.94 81.28 0)
+    (property "Price (5 boards)" "7.05" (at 154.94 81.28 0)
       (effects (font (size 1.27 1.27)) hide)
     )
+    (property "JLCPCB Part #" "C2988620" (at 154.94 81.28 0)
+      (effects (font (size 1.27 1.27)) hide)
+    )
+    (property "Price" "1.41" (at 154.94 81.28 0)
+      (effects (font (size 1.27 1.27)) hide)
+    )

Commit message: updated schematic and footprints
Parts:
- BT1: footprint Battery:BatteryHolder_Keystone_1042_1x18650 -> Library:18650_Holder_SMD
Changed lines of the file:
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@@
       (effects (font (size 1.27 1.27)) (justify left))
     )
-    (property "Footprint" "Battery:BatteryHolder_Keystone_1042_1x18650" (at 154.94 79.756 90)
+    (property "Footprint" "Library:18650_Holder_SMD" (at 154.94 79.756 90)
       (effects (font (size 1.27 1.27)) hide)
     )
