File: FullSchematic/Charging Module.kicad_sch (KiCad schematic)
At the start: 14 parts, among them J1 TP4056

Commit message: Confirmed part numbers and prices
Parts:
- C1, C2: footprint Library:CAPC1608X90N -> Capacitor_SMD:C_0603_1608Metric; Populate (none) -> Yes
- D1, J1, LEDcharge, Qrevpol: Populate (none) -> Yes
- R1: footprint Library:RESC2013X65N -> Resistor_SMD:R_1206_3216Metric; Populate (none) -> Yes; Price 0.001 -> 0.01; Price ( 1 board) 0.001 -> 0.01; Price (5 boards) 0.005 -> 0.05
- R15, R2, R4, R5: footprint Library:RESC2013X65N -> Resistor_SMD:R_1206_3216Metric; Populate (none) -> Yes
Changed lines of the file:
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@@
       (effects (font (size 1.27 1.27)) (justify left))
     )
-    (property "Footprint" "Library:CAPC1608X90N" (at 129.54 87.63 0)
+    (property "Footprint" "Capacitor_SMD:C_0603_1608Metric" (at 129.54 87.63 0)
       (effects (font (size 1.27 1.27)) hide)
     )
@@
     )
     (property "JLCPCB Part #" "C1691" (at 129.54 87.63 0)
+      (effects (font (size 1.27 1.27)) hide)
+    )
+    (property "Populate" "Yes" (at 129.54 87.63 0)
       (effects (font (size 1.27 1.27)) hide)
     )
@@
       (effects (font (size 1.27 1.27)) (justify left))
     )
-    (property "Footprint" "Library:CAPC1608X90N" (at 173.99 88.9 0)
+    (property "Footprint" "Capacitor_SMD:C_0603_1608Metric" (at 173.99 88.9 0)
       (effects (font (size 1.27 1.27)) hide)
     )
@@
       (effects (font (size 1.27 1.27)) hide)
     )
+    (property "Populate" "Yes" (at 173.99 88.9 0)
+      (effects (font (size 1.27 1.27)) hide)
+    )
     (pin "1")
     (pin "2")
@@
     )
     (property "JLCPCB Part #" "C437199" (at 109.22 78.74 0)
+      (effects (font (size 1.27 1.27)) hide)
+    )
+    (property "Populate" "Yes" (at 109.22 78.74 0)
       (effects (font (size 1.27 1.27)) hide)
     )
@@
       (effects (font (size 1 1)))
     )
-    (property "Footprint" "Library:RESC2013X65N" (at 134.62 73.66 0)
+    (property "Footprint" "Resistor_SMD:R_1206_3216Metric" (at 134.62 73.66 0)
       (effects (font (size 1.27 1.27)) hide)
     )
@@
       (effects (font (size 1.27 1.27)) hide)
     )
-    (property "Price" "0.001" (at 134.62 73.66 0)
-      (effects (font (size 1.27 1.27)) hide)
-    )
-    (property "Price ( 1 board)" "0.001" (at 134.62 73.66 0)
-      (effects (font (size 1.27 1.27)) hide)
-    )
-    (property "Price (5 boards)" "0.005" (at 134.62 73.66 0)
+    (property "Price" "0.01" (at 134.62 73.66 0)
+      (effects (font (size 1.27 1.27)) hide)
+    )
+    (property "Price ( 1 board)" "0.01" (at 134.62 73.66 0)
+      (effects (font (size 1.27 1.27)) hide)
+    )
+    (property "Price (5 boards)" "0.05" (at 134.62 73.66 0)
       (effects (font (size 1.27 1.27)) hide)
     )
@@
       (effects (font (size 1.27 1.27)) hide)
     )
+    (property "Populate" "Yes" (at 134.62 73.66 0)
+      (effects (font (size 1.27 1.27)) hide)
+    )
     (pin "1")
     (pin "2")
@@
     )
     (property "Price" "0.01" (at 190.5 73.66 0)
+      (effects (font (size 1.27 1.27)) hide)
+    )
+    (property "Populate" "Yes" (at 190.5 73.66 0)
       (effects (font (size 1.27 1.27)) hide)
     )
@@
       (effects (font (size 1.27 1.27)))
     )
-    (property "Footprint" "Library:RESC2013X65N" (at 205.994 98.806 90)
+    (property "Footprint" "Resistor_SMD:R_1206_3216Metric" (at 205.994 98.806 90)
       (effects (font (size 1.27 1.27)) hide)
     )
@@
     )
     (property "Price (5 boards)" "0.06" (at 207.01 99.06 0)
+      (effects (font (size 1.27 1.27)) hide)
+    )
+    (property "Populate" "Yes" (at 207.01 99.06 0)
       (effects (font (size 1.27 1.27)) hide)
     )
@@
     )
     (property "Price" "0.11" (at 138.43 71.12 0)
+      (effects (font (size 1.27 1.27)) hide)
+    )
+    (property "Populate" "Yes" (at 138.43 71.12 0)
       (effects (font (size 1.27 1.27)) hide)
     )
@@
       (effects (font (size 1.27 1.27)))
     )
-    (property "Footprint" "Library:RESC2013X65N" (at 195.834 81.534 90)
+    (property "Footprint" "Resistor_SMD:R_1206_3216Metric" (at 195.834 81.534 90)
       (effects (font (size 1.27 1.27)) hide)
     )
@@
     )
     (property "Price (5 boards)" "0.06" (at 195.58 82.55 0)
+      (effects (font (size 1.27 1.27)) hide)
+    )
+    (property "Populate" "Yes" (at 195.58 82.55 0)
       (effects (font (size 1.27 1.27)) hide)
     )
@@
       (effects (font (size 1.27 1.27)))
     )
-    (property "Footprint" "Library:RESC2013X65N" (at 181.61 73.66 0)
+    (property "Footprint" "Resistor_SMD:R_1206_3216Metric" (at 181.61 73.66 0)
       (effects (font (size 1.27 1.27)) hide)
     )
@@
       (effects (font (size 1.27 1.27)) hide)
     )
+    (property "Populate" "Yes" (at 181.61 73.66 0)
+      (effects (font (size 1.27 1.27)) hide)
+    )
     (pin "1")
     (pin "2")
@@
       (effects (font (size 1.27 1.27)))
     )
-    (property "Footprint" "Library:RESC2013X65N" (at 120.904 77.724 90)
+    (property "Footprint" "Resistor_SMD:R_1206_3216Metric" (at 120.904 77.724 90)
       (effects (font (size 1.27 1.27)) hide)
     )
@@
     )
     (property "Price (5 boards)" "0.06" (at 120.65 78.74 0)
+      (effects (font (size 1.27 1.27)) hide)
+    )
+    (property "Populate" "Yes" (at 120.65 78.74 0)
       (effects (font (size 1.27 1.27)) hide)
     )
@@
       (effects (font (size 1.27 1.27)) hide)
     )
+    (property "Populate" "Yes" (at 204.47 87.63 0)
+      (effects (font (size 1.27 1.27)) hide)
+    )

Commit message: Checked part #s, prices, footprints
Parts:
- added D1: Schottky - 0.21@1A, Library:Schottky Diode, symbol Diode:1N5819
- added J3: Conn_01x03_Pin, Connector_PinHeader_2.54mm:PinHeader_1x03_P2.54mm_Vertical, symbol Connector:Conn_01x03_Pin
- C1, C2: Price 0.08 -> 0.0052; Price ( 1 board) 0.24 -> 0.0208; Price (5 boards) 1.20 -> 0.104
- D1: value 1N5819 -> Schottky - 0.21@1A; footprint Library:Temp Schottky -> Library:Schottky Diode; JLCPCB Part # C437199 -> C413465; Price 0.0167 -> 0.20; Price ( 1 board) 0.0167 -> 0.4; Price (5 boards) 0.0835 -> 2
- LEDcharge: footprint LED_THT:LED_D3.0mm_IRBlack -> LED_SMD:LED_0603_1608Metric
- Qrevpol: Price 0.09 -> 0.0721; Price ( 1 board) 0.18 -> 0.1442; Price (5 boards) 0.9 -> 0.721
- R15, R4, R5: Price ( 1 board) 0.012 -> 0.018; Price (5 boards) 0.06 -> 0.09
- R2: Price 0.001 -> 0.003; Price ( 1 board) 0.001 -> 0.003; Price (5 boards) 0.005 -> 0.015
Connections:
- net Vbat: now also J3.2 (Pin_2); no longer R4.1, TP15.1
- net at Qrevpol.1 (D), R15.2: now also D1.2 (A)
- new net: J3.1 (Pin_1), R4.1, TP15.1
- new net: D1.1 (K), J3.3 (Pin_3)
Other:
- note added: "Redundant reverse polarity diode in case PMOS doesn't work"

Commit message: generated files
Parts:
- J3, TP15, TP16, TP19: JLCPCB Part # N/A -> (none)
Changed lines of the file:
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@@
       (effects (font (size 1.27 1.27)) hide)
     )
-    (property "JLCPCB Part #" "N/A" (at 137.16 78.74 0)
+    (property "JLCPCB Part #" "" (at 137.16 78.74 0)
       (effects (font (size 1.27 1.27)) hide)
     )
@@
       (effects (font (size 1.27 1.27)) hide)
     )
-    (property "JLCPCB Part #" "N/A" (at 240.03 111.76 0)
+    (property "JLCPCB Part #" "" (at 240.03 111.76 0)
       (effects (font (size 1.27 1.27)) hide)
     )
@@
       (effects (font (size 1.27 1.27)) hide)
     )
-    (property "JLCPCB Part #" "N/A" (at 207.01 105.41 0)
+    (property "JLCPCB Part #" "" (at 207.01 105.41 0)
       (effects (font (size 1.27 1.27)) hide)
     )
@@
       (effects (font (size 1.27 1.27)) hide)
     )
-    (property "JLCPCB Part #" "N/A" (at 181.61 82.55 0)
-      (effects (font (size 1.27 1.27)) hide)
-    )
+    (property "JLCPCB Part #" "" (at 181.61 82.55 0)
+      (effects (font (size 1.27 1.27)) hide)
+    )

Commit message: Decreased Price
Parts:
- C1, C2: footprint Capacitor_SMD:C_0603_1608Metric -> Capacitor_SMD:C_1206_3216Metric; JLCPCB Part # C1691 -> C13585
- Qrevpol: JLCPCB Part # C5337196 -> C10487
Changed lines of the file:
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@@
       (effects (font (size 1.27 1.27)) (justify left))
     )
-    (property "Footprint" "Capacitor_SMD:C_0603_1608Metric" (at 129.54 87.63 0)
+    (property "Footprint" "Capacitor_SMD:C_1206_3216Metric" (at 129.54 87.63 0)
       (effects (font (size 1.27 1.27)) hide)
     )
@@
       (effects (font (size 1.27 1.27)) hide)
     )
-    (property "JLCPCB Part #" "C1691" (at 129.54 87.63 0)
+    (property "JLCPCB Part #" "C13585" (at 129.54 87.63 0)
       (effects (font (size 1.27 1.27)) hide)
     )
@@
       (effects (font (size 1.27 1.27)) (justify left))
     )
-    (property "Footprint" "Capacitor_SMD:C_0603_1608Metric" (at 173.99 88.9 0)
+    (property "Footprint" "Capacitor_SMD:C_1206_3216Metric" (at 173.99 88.9 0)
       (effects (font (size 1.27 1.27)) hide)
     )
@@
       (effects (font (size 1.27 1.27)) hide)
     )
-    (property "JLCPCB Part #" "C1691" (at 173.99 88.9 0)
+    (property "JLCPCB Part #" "C13585" (at 173.99 88.9 0)
       (effects (font (size 1.27 1.27)) hide)
     )
@@
       (effects (font (size 1.27 1.27)) hide)
     )
-    (property "JLCPCB Part #" "C5337196" (at 204.47 87.63 0)
-      (effects (font (size 1.27 1.27)) hide)
-    )
+    (property "JLCPCB Part #" "C10487" (at 204.47 87.63 0)
+      (effects (font (size 1.27 1.27)) hide)
+    )
