File: FullSchematic/FullSchematic.kicad_pcb (KiCad board)
At the start: 2 copper layers, 100 x 100 mm, 85 parts, among them IC1 TTP223E-BA6, J1 USB_B_Micro, J2 TP4056, J3 Conn_01x03_Pin, J4 Conn_01x03_Pin, J5 Conn_01x03_Pin, P1 Touch Pad, Q1 IRLML6402, Q2 IRLML6402, Q3 IRLML6402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

Commit message: Decreased Price
Parts:
- C10, C11, C8, C9: footprint Capacitor_SMD:C_0603_1608Metric -> Capacitor_SMD:C_1206_3216Metric
- C13: footprint Capacitor_THT:C_Disc_D4.3mm_W1.9mm_P5.00mm -> Capacitor_SMD:C_1206_3216Metric
- D5: footprint LED_SMD:LED_0201_0603Metric -> LED_SMD:LED_0805_2012Metric
- Q1, Q2, Q3: value IRLML6402 -> SI2301CDS
- R1, R2, R3: footprint Resistor_SMD:R_1206_3216Metric -> Resistor_SMD:R_0805_2012Metric
- U1: value LM1117-3.3 -> XC6206P332MR; footprint Package_TO_SOT_SMD:SOT-223 -> Package_TO_SOT_SMD:SOT-23-3
- U3: value 24LC64 -> AT24C256C
- U5: value OP184 -> NE5532
- moved C13 0.97 mm to (108.2, 94.2), turned to -90 degrees
- moved C9 0.81 mm to (73.3, 141.6)
- moved D5 0.65 mm to (113.6, 98.7)
Connections:
- C9 pad 1: Net-(U1-VO) -> Net-(U1-VI)
- R17 pad 1: Net-(U1-VO) -> Net-(U1-VI)
- U1 pad 2: Net-(U1-VO) -> /Power Module/Regulating/Vin
- U1 pad 3: /Power Module/Regulating/Vin -> Net-(U1-VI)
- U5 pad 1: unconnected-(U5-VOS-Pad1) -> Net-(R14-Pad2)
- U5 pad 6: Net-(R14-Pad2) -> unconnected-(U5-Pad6)
- U5 pad 7: /Power Module/Charging/Vbat -> unconnected-(U5-V+-Pad7)
- U5 pad 8: unconnected-(U5-VOS-Pad8) -> /Power Module/Charging/Vbat
Routing:
- net Net-(U1-VI): track 0.00 -> 13.4 mm
- net Net-(U1-VO): track 9.89 -> 0.00 mm
- net Net-(R14-Pad2): track 51.2 -> 58.6 mm, vias 4 -> 6
- net /Power Module/Regulating/Vin: track 29.7 -> 32.2 mm
- net GND: track 104.0 -> 106.2 mm
- net /Power Module/Charging/Vbat: track 101.6 -> 100.3 mm
- net Net-(D5-A): track 5.34 -> 4.41 mm
- net /Vboard: track 247.2 -> 246.5 mm
