File: FullSchematic/FullSchematic.kicad_pcb (KiCad board)
At the start: 2 copper layers, 100 x 100 mm, 85 parts, among them IC1 TTP223E-BA6, J1 USB_B_Micro, J2 TP4056, J3 Conn_01x03_Pin, J4 Conn_01x03_Pin, J5 Conn_01x03_Pin, P1 Touch Pad, Q1 SI2301CDS, Q2 SI2301CDS, Q3 SI2301CDS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

Commit message: Uploaded final board design
Parts:
- removed U5: NE5532, Library:SOIC127P600X175-8N
- added G***: LOGO, Library:ManUtd, B.Cu at (102.5, 64.8)
- added R24: 4.7k, Library:RESC2013X65N, F.Cu at (115.2, 133.5)
- added U7: NE5532, Package_SO:SOIC-8_3.9x4.9mm_P1.27mm, F.Cu at (91.3, 98.9)
- C5: footprint Capacitor_THT:C_Disc_D4.7mm_W2.5mm_P5.00mm -> Capacitor_SMD:C_0805_2012Metric
- J3: value Conn_01x03_Pin -> Conn_01x04_Pin; footprint Connector_PinHeader_2.54mm:PinHeader_1x03_P2.54mm_Vertical -> Connector_PinHeader_2.54mm:PinHeader_1x04_P2.54mm_Vertical
- R11: value 180 -> 10k
- R6: value 4700 -> 4.7k
- moved C5 3.70 mm to (113.5, 93.9)
- moved J3 0.60 mm to (147.6, 105.0)
- moved R6 0.15 mm to (128.4, 127.4), turned to 180 degrees
Connections:
- C9 pad 1: Net-(U1-VI) -> Net-(U1-VO)
- J3 pad 1: /Pin 1 -> /Microcontroller/T_sensor
- J3 pad 2: /Microcontroller/3.3V -> /Pin 2
- J3 pad 3: /Vboard -> /Microcontroller/3.3V
- Q1 pad 3: /Pin 1 -> /Pin 2
- R17 pad 1: Net-(U1-VI) -> Net-(U1-VO)
- R6 pad 1: /Microcontroller/SCL -> /Microcontroller/3.3V
- R6 pad 2: /Microcontroller/3.3V -> /Microcontroller/SDA
- TP17 pad 1: /Output of Touch Sensor -> /Microcontroller/T_sensor
- U1 pad 2: /Power Module/Regulating/Vin -> Net-(U1-VO)
- U1 pad 3: Net-(U1-VI) -> /Power Module/Regulating/Vin
- U3 pad 5: /Microcontroller/SCL -> /Microcontroller/SDA
- U4 pad 16: /Microcontroller/SCL -> /Microcontroller/SDA
- U4 pad 34: /Output of Touch Sensor -> /Microcontroller/T_sensor
Routing:
- net /Microcontroller/T_sensor: track 0.00 -> 64.5 mm, vias 0 -> 2
- net /Pin 1: track 48.6 -> 0.00 mm, vias 1 -> 0
- net /Pin 2: track 0.00 -> 47.8 mm, vias 0 -> 1
- net /Output of Touch Sensor: track 105.2 -> 61.1 mm
- net GND: track 106.2 -> 69.3 mm, vias 28 -> 6
- net /Microcontroller/3.3V: track 172.3 -> 199.2 mm, vias 3 -> 5
- net /Microcontroller/SDA: track 0.00 -> 21.6 mm
- net Net-(U1-VO): track 0.00 -> 15.4 mm
- net Net-(U6-K): track 42.2 -> 56.7 mm, vias 4 -> 2
- net Net-(U1-VI): track 13.4 -> 0.00 mm
- net /Microcontroller/LDR_sensor: track 85.2 -> 74.7 mm
- net /Power Module/Regulating/Vbat: track 99.7 -> 107.9 mm, vias 3 -> 5
- net /Power Module/Regulating/Vin: track 32.2 -> 40.4 mm
- net Net-(U7A--): track 16.7 -> 24.6 mm, vias 2 -> 4
- net Net-(Q1-G): track 14.0 -> 21.7 mm
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