File: FullSchematic/AnalogueSensor.kicad_sch (KiCad schematic)
At the start: 5 parts

Commit message: Confirmed part numbers and prices
Parts:
- R?: Populate yes -> Yes
- R?: footprint OptoDevice:R_LDR_10x8.5mm_P7.6mm_Vertical -> OptoDevice:R_LDR_5.0x4.1mm_P3mm_Vertical; Populate yes -> Yes
Changed lines of the file:
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@@
       (effects (font (size 1.27 1.27)) hide)
     )
-    (property "Populate" "yes" (at 81.28 58.42 0)
+    (property "Populate" "Yes" (at 81.28 58.42 0)
       (effects (font (size 1.27 1.27)) hide)
     )
@@
       (effects (font (size 1.27 1.27)) (justify left))
     )
-    (property "Footprint" "OptoDevice:R_LDR_10x8.5mm_P7.6mm_Vertical" (at 85.725 78.74 90)
+    (property "Footprint" "OptoDevice:R_LDR_5.0x4.1mm_P3mm_Vertical" (at 85.725 78.74 90)
       (effects (font (size 1.27 1.27)) hide)
     )
@@
       (effects (font (size 1.27 1.27)) hide)
     )
-    (property "Populate" "yes" (at 81.28 78.74 0)
+    (property "Populate" "Yes" (at 81.28 78.74 0)
       (effects (font (size 1.27 1.27)) hide)
     )

Commit message: generated files
Parts:
- TP10, TP8, TP9: JLCPCB Part # N/A -> (none)
Changed lines of the file:
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@@
       (effects (font (size 1.27 1.27)) hide)
     )
-    (property "JLCPCB Part #" "N/A" (at 81.28 63.5 0)
+    (property "JLCPCB Part #" "" (at 81.28 63.5 0)
       (effects (font (size 1.27 1.27)) hide)
     )
@@
       (effects (font (size 1.27 1.27)) hide)
     )
-    (property "JLCPCB Part #" "N/A" (at 81.28 72.39 0)
+    (property "JLCPCB Part #" "" (at 81.28 72.39 0)
       (effects (font (size 1.27 1.27)) hide)
     )
@@
       (effects (font (size 1.27 1.27)) hide)
     )
-    (property "JLCPCB Part #" "N/A" (at 92.71 68.58 0)
+    (property "JLCPCB Part #" "" (at 92.71 68.58 0)
       (effects (font (size 1.27 1.27)) hide)
     )

Commit message: Uploaded final board design
Parts:
- R?: value 180 -> 10k; JLCPCB Part # C22828 -> C25804
Changed lines of the file:
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@@
       (effects (font (size 1.27 1.27)) (justify left))
     )
-    (property "Value" "180" (at 82.7786 59.563 0)
+    (property "Value" "10k" (at 82.7786 59.563 0)
       (effects (font (size 1.27 1.27)) (justify left))
     )
@@
       (effects (font (size 1.27 1.27)) hide)
     )
-    (property "JLCPCB Part #" "C22828" (at 81.28 58.42 0)
+    (property "JLCPCB Part #" "C25804" (at 81.28 58.42 0)
       (effects (font (size 1.27 1.27)) hide)
     )
