File: FullSchematic/Microcontroller Schematic.kicad_sch (KiCad schematic)
At the start: 23 parts, among them J1 USB_B_Micro, J4 Conn_01x03_Pin, U2 CH340C, U3 AT24C256C, U4 STM32F051C6T6

Commit message: Uploaded final board design
Parts:
- added R24: 4.7k, Library:RESC2013X65N, symbol Device:R_US
- R6: value 4700 -> 4.7k
Connections:
- net SCL: now also R24.2; no longer R6.1, U3.5 (SDA), U4.16 (PA6)
- net Vboard: now also R6.1, R24.1; no longer R6.2
- new net SDA: R6.2, U3.5 (SDA), U4.16 (PA6)
Changed lines of the file:
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@@
 (kicad_sch (version 20230121) (generator eeschema)
   (paper "A4")
-  (junction (at 87.249 46.101) (diameter 0) (color 0 0 0 0)
-  )
   (junction (at 77.089 58.801) (diameter 0) (color 0 0 0 0)
   )
@@
   )
   (junction (at 95.123 97.663) (diameter 0) (color 0 0 0 0)
-  )
-  (junction (at 99.949 46.101) (diameter 0) (color 0 0 0 0)
   )
   (junction (at 87.249 51.181) (diameter 0) (color 0 0 0 0)
@@
     (stroke (width 0) (type default))
   )
-  (wire (pts (xy 112.649 42.291) (xy 99.949 42.291))
+  (wire (pts (xy 104.648 57.785) (xy 104.648 58.801))
     (stroke (width 0) (type default))
   )
@@
     (stroke (width 0) (type default))
   )
-  (wire (pts (xy 99.949 48.641) (xy 107.569 48.641))
-    (stroke (width 0) (type default))
-  )
-  (wire (pts (xy 97.409 58.801) (xy 101.219 58.801))
-    (stroke (width 0) (type default))
-  )
   (wire (pts (xy 195.453 36.703) (xy 195.453 39.243))
     (stroke (width 0) (type default))
   )
-  (wire (pts (xy 99.949 42.291) (xy 99.949 46.101))
-    (stroke (width 0) (type default))
-  )
   (wire (pts (xy 139.065 70.104) (xy 139.065 70.231))
     (stroke (width 0) (type default))
   )
-  (wire (pts (xy 87.249 46.101) (xy 89.789 46.101))
-    (stroke (width 0) (type default))
-  )
   (wire (pts (xy 97.663 102.743) (xy 97.663 97.663))
     (stroke (width 0) (type default))
@@
     (stroke (width 0) (type default))
   )
-  (wire (pts (xy 87.249 46.101) (xy 87.249 51.181))
+  (wire (pts (xy 87.249 42.291) (xy 87.249 51.181))
     (stroke (width 0) (type default))
   )
@@
     (stroke (width 0) (type default))
   )
-  (wire (pts (xy 97.409 46.101) (xy 99.949 46.101))
-    (stroke (width 0) (type default))
-  )
   (wire (pts (xy 210.693 31.242) (xy 190.5 31.242))
     (stroke (width 0) (type default))
@@
     (stroke (width 0) (type default))
   )
+  (wire (pts (xy 97.409 58.801) (xy 104.648 58.801))
+    (stroke (width 0) (type default))
+  )
   (wire (pts (xy 208.153 36.703) (xy 210.693 36.703))
     (stroke (width 0) (type default))
@@
     (stroke (width 0) (type default))
   )
+  (wire (pts (xy 116.078 57.912) (xy 116.078 61.341))
+    (stroke (width 0) (type default))
+  )
   (wire (pts (xy 181.483 112.903) (xy 190.373 112.903))
     (stroke (width 0) (type default))
@@
     (stroke (width 0) (type default))
   )
+  (wire (pts (xy 97.409 61.341) (xy 116.078 61.341))
+    (stroke (width 0) (type default))
+  )
   (wire (pts (xy 176.403 58.293) (xy 200.533 58.293))
     (stroke (width 0) (type default))
@@
     (stroke (width 0) (type default))
   )
-  (wire (pts (xy 87.249 42.291) (xy 87.249 46.101))
-    (stroke (width 0) (type default))
-  )
   (wire (pts (xy 93.853 171.958) (xy 93.853 176.403))
     (stroke (width 0) (type default))
@@
     (stroke (width 0) (type default))
   )
-  (wire (pts (xy 97.409 61.341) (xy 101.219 61.341))
-    (stroke (width 0) (type default))
-  )
   (wire (pts (xy 195.453 36.703) (xy 208.153 36.703))
     (stroke (width 0) (type default))
@@
     (stroke (width 0) (type default))
   )
+  (wire (pts (xy 116.078 50.292) (xy 116.078 47.752))
+    (stroke (width 0) (type default))
+  )
   (wire (pts (xy 77.089 58.801) (xy 77.089 51.181))
     (stroke (width 0) (type default))
@@
     (stroke (width 0) (type default))
   )
+  (wire (pts (xy 104.648 50.165) (xy 104.648 47.625))
+    (stroke (width 0) (type default))
+  )
   (wire (pts (xy 139.192 70.104) (xy 148.336 70.104))
     (stroke (width 0) (type default))
@@
   )
   (wire (pts (xy 163.703 112.903) (xy 170.053 112.903))
-    (stroke (width 0) (type default))
-  )
-  (wire (pts (xy 99.949 48.641) (xy 99.949 46.101))
     (stroke (width 0) (type default))
   )
@@
     (effects (font (size 1.27 1.27)) (justify left bottom))
   )
-  (label "SCL" (at 107.569 48.641 180) (fields_autoplaced)
-    (effects (font (size 1.27 1.27)) (justify right bottom))
-  )
   (label "SDA" (at 101.219 58.801 180) (fields_autoplaced)
     (effects (font (size 1.27 1.27)) (justify right bottom))
@@
     (effects (font (size 1.27 1.27)) (justify left bottom))
   )
-  (label "SDA" (at 112.649 42.291 180) (fields_autoplaced)
-    (effects (font (size 1.27 1.27)) (justify right bottom))
-  )
   (label "3.3V" (at 180.34 28.702 0) (fields_autoplaced)
     (effects (font (size 1.27 1.27)) (justify left bottom))
@@
     (effects (font (size 1.27 1.27)) (justify right))
   )
+  (hierarchical_label "Vboard" (shape input) (at 104.648 47.625 90) (fields_autoplaced)
+    (effects (font (size 1.27 1.27)) (justify left))
+  )
   (hierarchical_label "Vboard" (shape input) (at 115.443 104.013 90) (fields_autoplaced)
     (effects (font (size 1.27 1.27)) (justify left))
@@
   (hierarchical_label "T_sensor" (shape input) (at 70.358 161.163 180) (fields_autoplaced)
     (effects (font (size 1.27 1.27)) (justify right))
+  )
+  (hierarchical_label "Vboard" (shape input) (at 116.078 47.752 90) (fields_autoplaced)
+    (effects (font (size 1.27 1.27)) (justify left))
   )
   (symbol (lib_id "Device:LED") (at 194.183 130.683 180) (unit 1)
@@
     )
   )
+  (symbol (lib_id "Device:R_US") (at 116.078 54.102 0) (unit 1)
+    (in_bom yes) (on_board yes) (dnp no) (fields_autoplaced)
+    (property "Reference" "R24" (at 118.11 53.467 0)
+      (effects (font (size 1.27 1.27)) (justify left))
+    )
+    (property "Value" "4.7k" (at 118.11 56.007 0)
+      (effects (font (size 1.27 1.27)) (justify left))
+    )
+    (property "Footprint" "Library:RESC2013X65N" (at 117.094 54.356 90)
+      (effects (font (size 1.27 1.27)) hide)
+    )
+    (property "Datasheet" "~" (at 116.078 54.102 0)
+      (effects (font (size 1.27 1.27)) hide)
+    )
+    (property "Price" "0.001" (at 116.078 54.102 0)
+      (effects (font (size 1.27 1.27)) hide)
+    )
+    (property "Price ( 1 board)" "0.001" (at 116.078 54.102 0)
+      (effects (font (size 1.27 1.27)) hide)
+    )
+    (property "Price (5 boards)" "0.005" (at 116.078 54.102 0)
+      (effects (font (size 1.27 1.27)) hide)
+    )
+    (property "JLCPCB Part #" "C23162" (at 116.078 54.102 0)
+      (effects (font (size 1.27 1.27)) hide)
+    )
+    (property "Populate" "Yes" (at 116.078 54.102 0)
+      (effects (font (size 1.27 1.27)) hide)
+    )
+    (pin "1")
+    (pin "2")
+    (instances
+      (project "FullSchematic"
+        (path "/5dd86611-a33d-45ee-946c-01c599f30b12/5d08bf44-0550-4275-b6e8-e4566a125a74"
+          (reference "R24") (unit 1)
+        )
+      )
+      (project "Microcontroller Schematic"
+        (path "/87ad8a26-ca2b-40e6-a130-1e9e8587d367"
+          (reference "R6") (unit 1)
+        )
+      )
+    )
+  )
   (symbol (lib_id "power:GND") (at 201.803 130.683 0) (unit 1)
     (in_bom yes) (on_board yes) (dnp no) (fields_autoplaced)
@@
         (path "/5dd86611-a33d-45ee-946c-01c599f30b12/5d08bf44-0550-4275-b6e8-e4566a125a74"
           (reference "TP7") (unit 1)
+        )
+      )
+    )
+  )
+  (symbol (lib_id "Device:R_US") (at 104.648 53.975 0) (unit 1)
+    (in_bom yes) (on_board yes) (dnp no) (fields_autoplaced)
+    (property "Reference" "R6" (at 106.68 53.34 0)
+      (effects (font (size 1.27 1.27)) (justify left))
+    )
+    (property "Value" "4.7k" (at 106.68 55.88 0)
+      (effects (font (size 1.27 1.27)) (justify left))
+    )
+    (property "Footprint" "Library:RESC2013X65N" (at 105.664 54.229 90)
+      (effects (font (size 1.27 1.27)) hide)
+    )
+    (property "Datasheet" "~" (at 104.648 53.975 0)
+      (effects (font (size 1.27 1.27)) hide)
+    )
+    (property "Price" "0.001" (at 104.648 53.975 0)
+      (effects (font (size 1.27 1.27)) hide)
+    )
+    (property "Price ( 1 board)" "0.001" (at 104.648 53.975 0)
+      (effects (font (size 1.27 1.27)) hide)
+    )
+    (property "Price (5 boards)" "0.005" (at 104.648 53.975 0)
+      (effects (font (size 1.27 1.27)) hide)
+    )
+    (property "JLCPCB Part #" "C23162" (at 104.648 53.975 0)
+      (effects (font (size 1.27 1.27)) hide)
+    )
+    (property "Populate" "Yes" (at 104.648 53.975 0)
+      (effects (font (size 1.27 1.27)) hide)
+    )
+    (pin "1")
+    (pin "2")
+    (instances
+      (project "FullSchematic"
+        (path "/5dd86611-a33d-45ee-946c-01c599f30b12/5d08bf44-0550-4275-b6e8-e4566a125a74"
+          (reference "R6") (unit 1)
+        )
+      )
+      (project "Microcontroller Schematic"
+        (path "/87ad8a26-ca2b-40e6-a130-1e9e8587d367"
+          (reference "R6") (unit 1)
         )
       )
@@
         )
       )
-    )
-  )
-  (symbol (lib_id "Device:R_US") (at 93.599 46.101 270) (unit 1)
-    (in_bom yes) (on_board yes) (dnp no) (fields_autoplaced)
-    (property "Reference" "R6" (at 93.599 42.2021 90)
-      (effects (font (size 1.27 1.27)))
-    )
-    (property "Value" "4700" (at 93.599 44.1231 90)
-      (effects (font (size 1.27 1.27)))
-    )
-    (property "Footprint" "Library:RESC2013X65N" (at 93.345 47.117 90)
-      (effects (font (size 1.27 1.27)) hide)
-    )
-    (property "Datasheet" "~" (at 93.599 46.101 0)
-      (effects (font (size 1.27 1.27)) hide)
-    )
-    (property "Price" "0.001" (at 93.599 46.101 0)
-      (effects (font (size 1.27 1.27)) hide)
-    )
-    (property "Price ( 1 board)" "0.001" (at 93.599 46.101 0)
-      (effects (font (size 1.27 1.27)) hide)
-    )
-    (property "Price (5 boards)" "0.005" (at 93.599 46.101 0)
-      (effects (font (size 1.27 1.27)) hide)
-    )
-    (property "JLCPCB Part #" "C23162" (at 93.599 46.101 0)
-      (effects (font (size 1.27 1.27)) hide)
-    )
-    (property "Populate" "Yes" (at 93.599 46.101 0)
-      (effects (font (size 1.27 1.27)) hide)
-    )
-    (pin "1")
-    (pin "2")
-    (instances
-      (project "FullSchematic"
-        (path "/5dd86611-a33d-45ee-946c-01c599f30b12/5d08bf44-0550-4275-b6e8-e4566a125a74"
-          (reference "R6") (unit 1)
-        )
-      )
-      (project "Microcontroller Schematic"
-        (path "/87ad8a26-ca2b-40e6-a130-1e9e8587d367"
-          (reference "R6") (unit 1)
-        )
-      )
