File: FullSchematic/Power module.kicad_sch (KiCad schematic)
At the start: 16 parts, among them Q2 IRLML6402, U5 OP184, U6 CJ432

Commit message: Decreased Price
Parts:
- Q2: value IRLML6402 -> SI2301CDS; JLCPCB Part # C518785 -> C10487
- R14: JLCPCB Part # C416080 -> C17514
- R19: JLCPCB Part # C429049 -> C25755
- R21: JLCPCB Part # C465471 -> 0805
- R22, R8: JLCPCB Part # C465466 -> C22976
- U5: value OP184 -> NE5532; JLCPCB Part # C690879 -> C7426
Connections:
- net Charging/Vbat: now also U5.8 (VOS); no longer U5.7 (V+)
- net at U5.1 (VOS): now also R14.2, R18.1, TP18.1
- now unconnected: U5.6
Changed lines of the file:
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@@
   (junction (at 194.691 111.887) (diameter 0) (color 0 0 0 0)
   )
-  (junction (at 159.512 101.6) (diameter 0) (color 0 0 0 0)
-  )
   (junction (at 125.222 101.6) (diameter 0) (color 0 0 0 0)
   )
   (junction (at 145.669 111.252) (diameter 0) (color 0 0 0 0)
   )
+  (junction (at 165.354 101.6) (diameter 0) (color 0 0 0 0)
+  )
   (junction (at 194.691 121.666) (diameter 0) (color 0 0 0 0)
   )
@@
   (junction (at 129.54 101.6) (diameter 0) (color 0 0 0 0)
   )
+  (junction (at 154.94 119.126) (diameter 0) (color 0 0 0 0)
+  )
   (junction (at 208.534 127.254) (diameter 0) (color 0 0 0 0)
   )
@@
   (junction (at 208.534 111.125) (diameter 0) (color 0 0 0 0)
   )
-  (junction (at 154.94 119.126) (diameter 0) (color 0 0 0 0)
-  )
   (junction (at 208.534 109.22) (diameter 0) (color 0 0 0 0)
   )
@@
   (junction (at 194.691 130.302) (diameter 0) (color 0 0 0 0)
   )
-  (no_connect (at 172.847 111.506))
-  (no_connect (at 170.307 111.506))
+  (no_connect (at 175.387 126.746))
+  (no_connect (at 165.227 119.126))
   (wire (pts (xy 208.534 101.6) (xy 208.534 104.14))
     (stroke (width 0) (type default))
   )
+  (wire (pts (xy 172.847 110.236) (xy 172.847 111.506))
+    (stroke (width 0) (type default))
+  )
   (wire (pts (xy 194.691 111.887) (xy 194.691 112.014))
     (stroke (width 0) (type default))
@@
     (stroke (width 0) (type default))
   )
+  (wire (pts (xy 165.354 101.6) (xy 194.691 101.6))
+    (stroke (width 0) (type default))
+  )
   (wire (pts (xy 194.691 121.666) (xy 194.691 123.19))
     (stroke (width 0) (type default))
   )
+  (wire (pts (xy 157.353 110.236) (xy 157.353 119.126))
+    (stroke (width 0) (type default))
+  )
   (wire (pts (xy 192.278 132.461) (xy 192.278 130.302))
     (stroke (width 0) (type default))
@@
     (stroke (width 0) (type default))
   )
-  (wire (pts (xy 150.749 101.6) (xy 159.512 101.6))
+  (wire (pts (xy 150.749 101.6) (xy 165.354 101.6))
+    (stroke (width 0) (type default))
+  )
+  (wire (pts (xy 154.94 119.126) (xy 157.353 119.126))
     (stroke (width 0) (type default))
   )
@@
     (stroke (width 0) (type default))
   )
-  (wire (pts (xy 154.94 119.126) (xy 165.227 119.126))
-    (stroke (width 0) (type default))
-  )
   (wire (pts (xy 145.669 111.252) (xy 145.669 111.379))
     (stroke (width 0) (type default))
@@
     (stroke (width 0) (type default))
   )
-  (wire (pts (xy 159.512 101.6) (xy 194.691 101.6))
+  (wire (pts (xy 165.354 111.506) (xy 165.354 101.6))
     (stroke (width 0) (type default))
   )
@@
     (stroke (width 0) (type default))
   )
+  (wire (pts (xy 170.307 111.506) (xy 165.354 111.506))
+    (stroke (width 0) (type default))
+  )
   (wire (pts (xy 109.22 119.38) (xy 104.14 119.38))
     (stroke (width 0) (type default))
   )
-  (wire (pts (xy 175.387 126.746) (xy 159.512 126.746))
-    (stroke (width 0) (type default))
-  )
   (wire (pts (xy 62.23 120.65) (xy 34.29 120.65))
     (stroke (width 0) (type default))
@@
     (stroke (width 0) (type default))
   )
-  (wire (pts (xy 159.512 126.746) (xy 159.512 101.6))
-    (stroke (width 0) (type default))
-  )
   (wire (pts (xy 208.534 111.125) (xy 208.534 111.252))
     (stroke (width 0) (type default))
@@
   )
   (wire (pts (xy 208.534 73.66) (xy 154.94 73.66))
+    (stroke (width 0) (type default))
+  )
+  (wire (pts (xy 157.353 110.236) (xy 172.847 110.236))
     (stroke (width 0) (type default))
   )
@@
       (effects (font (size 1.27 1.27)))
     )
-    (property "Value" "OP184" (at 162.56 117.4749 0)
+    (property "Value" "NE5532" (at 162.56 117.4749 0)
       (effects (font (size 1.27 1.27)))
     )
@@
       (effects (font (size 1.27 1.27)) hide)
     )
-    (property "JLCPCB Part #" "C690879" (at 172.847 119.126 0)
+    (property "JLCPCB Part #" "C7426" (at 172.847 119.126 0)
       (effects (font (size 1.27 1.27)) hide)
     )
@@
       (effects (font (size 1.27 1.27)) hide)
     )
-    (property "JLCPCB Part #" "C465466" (at 208.534 106.68 0)
+    (property "JLCPCB Part #" "C22976" (at 208.534 106.68 0)
       (effects (font (size 1.27 1.27)) hide)
     )
@@
       (effects (font (size 1.27 1.27)))
     )
-    (property "Value" "IRLML6402" (at 145.669 97.79 90)
+    (property "Value" "SI2301CDS" (at 145.669 97.79 90)
       (effects (font (size 1.27 1.27)))
     )
@@
       (effects (font (size 1.27 1.27)) (justify left) hide)
     )
-    (property "JLCPCB Part #" "C518785" (at 145.669 104.14 0)
+    (property "JLCPCB Part #" "C10487" (at 145.669 104.14 0)
       (effects (font (size 1.27 1.27)) hide)
     )
@@
       (effects (font (size 1.27 1.27)) hide)
     )
-    (property "JLCPCB Part #" "C416080" (at 145.669 113.792 0)
+    (property "JLCPCB Part #" "C17514" (at 145.669 113.792 0)
       (effects (font (size 1.27 1.27)) hide)
     )
@@
       (effects (font (size 1.27 1.27)) hide)
     )
-    (property "JLCPCB Part #" "C465466" (at 208.534 113.665 0)
+    (property "JLCPCB Part #" "C22976" (at 208.534 113.665 0)
       (effects (font (size 1.27 1.27)) hide)
     )
@@
       (effects (font (size 1.27 1.27)) hide)
     )
-    (property "JLCPCB Part #" "C465471" (at 125.222 116.078 0)
+    (property "JLCPCB Part #" "0805" (at 125.222 116.078 0)
       (effects (font (size 1.27 1.27)) hide)
     )
@@
       (effects (font (size 1.27 1.27)) hide)
     )
-    (property "JLCPCB Part #" "C429049" (at 194.691 132.842 0)
-      (effects (font (size 1.27 1.27)) hide)
-    )
+    (property "JLCPCB Part #" "C25755" (at 194.691 132.842 0)
+      (effects (font (size 1.27 1.27)) hide)
+    )

Commit message: Uploaded final board design
Parts:
- removed U5: NE5532, Library:SOIC127P600X175-8N, symbol Amplifier_Operational:OP07
- added U7: NE5532, Package_SO:SOIC-8_3.9x4.9mm_P1.27mm, symbol Amplifier_Operational:NE5532
Connections:
- net at R20.2, TP20.1, U6.1 (REF)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: now also U7.3 (+)
- net at R14.2, R18.1, TP18.1: now also U7.1
- net at R8.2, R9.1: now also U7.2 (-)
- no-connect marks 2 -> 0
