File: 1. Final Project/DigitalSensor.kicad_sch (KiCad schematic)
At the start: 10 parts, among them P1 Touch Pad

Commit message: made sure git repo is up to date
Parts:
- IC?: footprint Package_TO_SOT_SMD:SOT-563 -> Package_TO_SOT_SMD:SOT-23-6
Changed lines of the file:
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@@
       (effects (font (size 1.27 1.27)))
     )
-    (property "Footprint" "Package_TO_SOT_SMD:SOT-563" (at 162.56 92.71 0)
+    (property "Footprint" "Package_TO_SOT_SMD:SOT-23-6" (at 162.56 92.71 0)
       (effects (font (size 1.27 1.27)) (justify left) hide)
     )
