File: 1. Final Project/FullSchematic.kicad_pcb (KiCad board)
At the start: 2 copper layers, 100 x 100 mm, 87 parts, among them IC1 TTP223E-BA6, J1 USB_B_Micro, J2 TP4056, J3 Conn_01x04_Pin, J4 Conn_01x03_Pin, J5 Conn_01x03_Pin, P1 Touch Pad, Q1 SI2301CDS, Q2 SI2301CDS, Q3 SI2301CDS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

Commit message: made sure git repo is up to date
Parts:
- IC1: footprint Package_TO_SOT_SMD:SOT-563 -> Package_TO_SOT_SMD:SOT-23-6
- moved IC1 2.05 mm to (116.7, 85.6)
Routing:
- net /Output of Touch Sensor: track 61.1 -> 62.7 mm
